Commit message: fix caster radius to fix bounce

File: my_robot/urdf/my_robot.xacro (robot description, xacro)
@@ -31,8 +31,20 @@
         </geometry>
         </visual>
+        <collision name='back_caster_collision'>
+        <origin xyz="-0.15 0 -0.05" rpy=" 0 0 0"/>
+        <geometry>
+            <sphere radius="0.0299"/>
+        </geometry>
+        </collision>
+        <visual name='back_caster_visual'>
+        <origin xyz="-0.15 0 -0.05" rpy=" 0 0 0"/>
+        <geometry>
+            <sphere radius="0.0300"/>
+        </geometry>
+        </visual>
         <collision name='front_caster_collision'>
         <origin xyz="0.15 0 -0.05" rpy=" 0 0 0"/>
         <geometry>
-            <sphere radius="0.0324"/>
+            <sphere radius="0.0299"/>
         </geometry>
         </collision>
@@ -40,5 +52,5 @@
         <origin xyz="0.15 0 -0.05" rpy=" 0 0 0"/>
         <geometry>
-            <sphere radius="0.0325"/>
+            <sphere radius="0.0300"/>
         </geometry>
         </visual>
